File: IRRemo/IRRemo.sch (KiCad schematic (older format))
At the start: 16 parts, among them J1 Conn_01x05_Male, J2 Conn_02x02_Odd_Even, J3 Conn_01x03_Male, J4 Conn_01x02_Male, J5 Conn_01x02_Male, U1 CY8C4244, U2 GP1UXC41QS, U3 BD6211F, U4 BD6211F

Commit message: BGA
Parts:
- removed U1: CY8C4244, Package_SO:SSOP-28_5.3x10.2mm_P0.65mm, symbol CY8C4244:CY8C4244PVI-442
- added JP1, JP2: SolderJumper_2_Bridged, 2020-08-21_07-11-41:Jumper-Con, symbol Jumper:SolderJumper_2_Bridged
- added U1: CY8C4245FNI-483T, 2020-08-21_07-11-41:BGA35N35P7X5_258X209X48N, symbol CY8C4125FNI-S433T:CY8C4245FNI-483T
- J2: value Conn_02x02_Odd_Even -> SER
Connections:
- net +3V0: now also JP1.2 (B); no longer C1.1
- net GND: now also JP2.2 (B)
- net IR: now also U1.E5 (P2.4)
- net SWDCK: now also U1.C1 (P3.3)
- net SWDIO: now also U1.D1 (P3.2)
- net XRES: now also U1.B6 (XRES)
- net at U3.4 (FIN): now also U1.C3 (P0.0)
- net at U3.5 (RIN): now also U1.A5 (P0.1)
- net at U4.4 (FIN): now also U1.A4 (P0.2)
- net at U4.5 (RIN): now also U1.A3 (P0.3)
- net at C4.1: now also U1.A7 (VCCD)
- net at J3.1 (Pin_1): now also U1.B2 (P4.1)
- net at J3.2 (Pin_2): now also U1.B1 (P4.0)
- net at J2.3 (Pin_3): now also U1.E3 (P2.6)
- net at J2.1 (Pin_1): now also U1.E2 (P2.7)
- net at R1.2: now also D1.2 (A)
- net at R1.1: now also U1.E4 (P2.3); no longer D1.2 (A)
- new net VDD: C1.1, JP1.1 (A), U1.C7 (VDD)
- new net Vss: JP2.1 (A), U1.B7 (VSS)
Other:
- note added: "G\nR\nT"
- note added: "IR Remo v1.4"
- note removed: "G\nT\nR"
- note removed: "IR Remo v1.3"
- moved on the sheet: C1, C4, D1, J2, R1, U2
